File: PCB/Cargador RPi/Tarjeta RPi/Eagle/CargadorRPi/Cargador_RasPi3HAT_CamSlot_v2.0.brd (EAGLE design)
At the start: 65 x 56 mm, 26 parts, among them J2 PIN20X2, U1 MCP3208, X1 ZX62D-B-5PA8

Commit message: Ajuste en la ubicación del puerto micro USB
Connections:
- removed net N$10: JP4.1, JP5.2
- removed net N$9: JP4.2, JP5.4
- net VBUS: now also JP4.1, JP5.2
- net VLIPO: now also JP4.2, JP5.4
Routing:
- net VLIPO: track 51.1 -> 81.1 mm
- net N$9: track 30.0 -> 0.00 mm
- net N$10: track 25.8 -> 0.00 mm
- net VBUS: track 92.9 -> 118.7 mm
Changed lines of the file:
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@@
 <?xml version="1.0" encoding="utf-8"?>
 <!DOCTYPE eagle SYSTEM "eagle.dtd">
-<eagle version="9.3.0">
+<eagle version="9.3.2">
 <drawing>
 <settings>
-<setting alwaysvectorfont="yes"/>
+<setting alwaysvectorfont="no"/>
 <setting keepoldvectorfont="yes"/>
 <setting verticaltext="up"/>
@@
 <wire x1="10" y1="16.1" x2="10" y2="2.65" width="1.016" layer="16"/>
 <wire x1="2.03" y1="18.32" x2="3.35" y2="17" width="1.016" layer="16"/>
+<contactref element="JP5" pad="2"/>
+<contactref element="JP4" pad="1"/>
+<wire x1="2" y1="31.11" x2="2" y2="24.7" width="1.016" layer="16"/>
+<wire x1="2" y1="24.7" x2="3.35" y2="23.35" width="1.016" layer="16"/>
+<wire x1="3.35" y1="23.35" x2="17" y2="23.35" width="1.016" layer="16"/>
+<wire x1="17" y1="23.35" x2="17.95" y2="22.4" width="1.016" layer="16"/>
+<wire x1="17.95" y1="22.4" x2="17.95" y2="19.94" width="1.016" layer="16"/>
+<wire x1="17.95" y1="19.94" x2="17.93" y2="19.92" width="0.1524" layer="16"/>
+<wire x1="17.93" y1="17.38" x2="17.93" y2="19.92" width="0" layer="19" extent="1-1"/>
 </signal>
 <signal name="VLIPO">
@@
 <wire x1="26.7" y1="3.65" x2="29.75" y2="3.65" width="1.016" layer="16"/>
 <wire x1="20.47" y1="11.63" x2="21.65" y2="10.45" width="1.016" layer="16"/>
+<contactref element="JP4" pad="2"/>
+<contactref element="JP5" pad="4"/>
+<wire x1="2" y1="33.65" x2="4.25" y2="33.65" width="1.016" layer="16"/>
+<wire x1="4.25" y1="33.65" x2="5.05" y2="32.85" width="1.016" layer="16"/>
+<wire x1="5.05" y1="32.85" x2="5.05" y2="27.2" width="1.016" layer="16"/>
+<wire x1="5.05" y1="27.2" x2="6.6" y2="25.65" width="1.016" layer="16"/>
+<wire x1="6.6" y1="25.65" x2="19" y2="25.65" width="1.016" layer="16"/>
+<wire x1="20.47" y1="24.18" x2="20.47" y2="19.92" width="1.016" layer="16"/>
+<wire x1="19" y1="25.65" x2="20.47" y2="24.18" width="1.016" layer="16"/>
+<wire x1="20.47" y1="19.92" x2="20.47" y2="17.38" width="0" layer="19" extent="1-1"/>
 </signal>
 <signal name="N$17">
@@
 <wire x1="5.825" y1="12" x2="4.57" y2="20.05" width="0" layer="19" extent="1-1"/>
 </signal>
-<signal name="N$9">
-<contactref element="JP4" pad="2"/>
-<contactref element="JP5" pad="4"/>
-<wire x1="2" y1="33.65" x2="4.25" y2="33.65" width="1.016" layer="16"/>
-<wire x1="4.25" y1="33.65" x2="5.05" y2="32.85" width="1.016" layer="16"/>
-<wire x1="5.05" y1="32.85" x2="5.05" y2="27.2" width="1.016" layer="16"/>
-<wire x1="5.05" y1="27.2" x2="6.6" y2="25.65" width="1.016" layer="16"/>
-<wire x1="6.6" y1="25.65" x2="19" y2="25.65" width="1.016" layer="16"/>
-<wire x1="20.47" y1="24.18" x2="20.47" y2="19.92" width="1.016" layer="16"/>
-<wire x1="19" y1="25.65" x2="20.47" y2="24.18" width="1.016" layer="16"/>
-</signal>
-<signal name="N$10">
-<contactref element="JP5" pad="2"/>
-<contactref element="JP4" pad="1"/>
-<wire x1="2" y1="31.11" x2="2" y2="24.7" width="1.016" layer="16"/>
-<wire x1="2" y1="24.7" x2="3.35" y2="23.35" width="1.016" layer="16"/>
-<wire x1="3.35" y1="23.35" x2="17" y2="23.35" width="1.016" layer="16"/>
-<wire x1="17" y1="23.35" x2="17.95" y2="22.4" width="1.016" layer="16"/>
-<wire x1="17.95" y1="22.4" x2="17.95" y2="19.94" width="1.016" layer="16"/>
-<wire x1="17.95" y1="19.94" x2="17.93" y2="19.92" width="0.1524" layer="16"/>
-</signal>
 </signals>
