File: PCB/Cargador RPi/Tarjeta RPi/Eagle/CargadorRPi/Cargador_RasPi3HAT_CamSlot_v2.0.sch (EAGLE design)
At the start: 26 parts, among them J2 PIN20X2, U1 MCP3208, X1 ZX62D-B-5PA8

Commit message: Se mejoran algunas pistas del PCB
Connections:
- removed net NC: J2.7, JP1.4
Changed lines of the file:
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@@
-</segment>
-</net>
-<net name="NC" class="0">
-<segment>
-<pinref part="JP1" gate="A" pin="4"/>
-<wire x1="30.48" y1="147.32" x2="22.86" y2="147.32" width="0.1524" layer="91"/>
-<label x="22.86" y="147.32" size="1.778" layer="95"/>
-<pinref part="J2" gate="G$1" pin="7"/>
-<wire x1="40.64" y1="147.32" x2="30.48" y2="147.32" width="0.1524" layer="91"/>
-<junction x="30.48" y="147.32"/>
 </segment>
 </net>

Commit message: Ajuste en la ubicación del puerto micro USB
Connections:
- removed net N$10: JP4.1, JP5-1.2
- removed net N$9: JP4.2, JP5-2.2
- net VBUS: now also JP4.1, JP5-1.2
- net VLIPO: now also JP4.2, JP5-2.2
Changed lines of the file:
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@@
 <?xml version="1.0" encoding="utf-8"?>
 <!DOCTYPE eagle SYSTEM "eagle.dtd">
-<eagle version="9.3.0">
+<eagle version="9.3.2">
 <drawing>
 <settings>
@@
 <wire x1="190.5" y1="228.6" x2="182.88" y2="228.6" width="0.1524" layer="91"/>
 </segment>
+<segment>
+<pinref part="JP5" gate="-1" pin="2"/>
+<wire x1="210.82" y1="215.9" x2="223.52" y2="215.9" width="0.1524" layer="91"/>
+<wire x1="223.52" y1="215.9" x2="223.52" y2="210.82" width="0.1524" layer="91"/>
+<pinref part="JP4" gate="A" pin="1"/>
+<wire x1="223.52" y1="210.82" x2="231.14" y2="210.82" width="0.1524" layer="91"/>
+<label x="193.04" y="215.9" size="1.778" layer="95"/>
+</segment>
 </net>
 <net name="VLIPO" class="0">
@@
 <wire x1="205.74" y1="205.74" x2="193.04" y2="205.74" width="0.1524" layer="91"/>
 </segment>
+<segment>
+<pinref part="JP4" gate="A" pin="2"/>
+<wire x1="228.6" y1="205.74" x2="231.14" y2="208.28" width="0.1524" layer="91"/>
+<pinref part="JP5" gate="-2" pin="2"/>
+<wire x1="208.28" y1="205.74" x2="228.6" y2="205.74" width="0.1524" layer="91"/>
+<label x="193.04" y="205.74" size="1.778" layer="95"/>
+</segment>
 </net>
 <net name="N$17" class="0">
@@
 </segment>
 </net>
-<net name="N$9" class="0">
-<segment>
-<pinref part="JP4" gate="A" pin="2"/>
-<wire x1="228.6" y1="205.74" x2="231.14" y2="208.28" width="0.1524" layer="91"/>
-<pinref part="JP5" gate="-2" pin="2"/>
-<wire x1="208.28" y1="205.74" x2="228.6" y2="205.74" width="0.1524" layer="91"/>
-</segment>
-</net>
-<net name="N$10" class="0">
-<segment>
-<pinref part="JP5" gate="-1" pin="2"/>
-<wire x1="210.82" y1="215.9" x2="223.52" y2="215.9" width="0.1524" layer="91"/>
-<wire x1="223.52" y1="215.9" x2="223.52" y2="210.82" width="0.1524" layer="91"/>
-<pinref part="JP4" gate="A" pin="1"/>
-<wire x1="223.52" y1="210.82" x2="231.14" y2="210.82" width="0.1524" layer="91"/>
-</segment>
-</net>
